Commit message: two agent also working

File: launch/opp_racecar.xacro (robot description, xacro)
@@ -11,4 +11,5 @@
   <xacro:property name="laser_height" value="0.05" />
   <xacro:property name="laser_radius" value="0.026" />
+  <xacro:property name="car_name" value="opp_racecar" />
   <material name="black">
     <color rgba="0.2 0.2 0.2 1."/>
@@ -17,7 +18,7 @@
     <color rgba="1. 0.57 0.1 1."/>
   </material>
-  <link name="base_link">
+  <link name="${car_name}/base_link">
     <visual>
-      <origin xyz="-0.1 0 ${ground_offset+height/2}"/>
+      <origin xyz="${wheelbase/2} 0 ${ground_offset+height/2}"/>
       <geometry>
         <box size="${wheelbase} ${width} ${height}"/>
@@ -27,9 +28,9 @@
   </link>
   <joint name="base_to_laser_model" type="fixed">
-    <parent link="base_link"/>
-    <child link="laser_model"/>
-    <origin xyz="0 0 ${ground_offset+height+(laser_height/2)}"/>
+    <parent link="${car_name}/base_link"/>
+    <child link="${car_name}/laser_model"/>
+    <origin xyz="${laser_distance_from_base_link} 0 ${ground_offset+height+(laser_height/2)}"/>
   </joint>
-  <link name="laser_model">
+  <link name="${car_name}/laser_model">
     <visual>
       <geometry>
@@ -39,10 +40,10 @@
     </visual>
   </link>
-  <joint name="base_to_back_left_wheel" type="fixed">
-    <parent link="base_link"/>
-    <child link="back_left_wheel"/>
-    <origin xyz="${-wheelbase/2-0.1} ${(wheel_length+width)/2} ${wheel_radius}"/>
+  <joint name="$base_to_back_left_wheel" type="fixed">
+    <parent link="${car_name}/base_link"/>
+    <child link="${car_name}/back_left_wheel"/>
+    <origin xyz="0 ${(wheel_length+width)/2} ${wheel_radius}"/>
   </joint>
-  <link name="back_left_wheel">
+  <link name="${car_name}/back_left_wheel">
     <visual>
       <geometry>
@@ -54,9 +55,9 @@
   </link>
   <joint name="base_to_back_right_wheel" type="fixed">
-    <parent link="base_link"/>
-    <child link="back_right_wheel"/>
-    <origin xyz="${-wheelbase/2-0.1} ${-(wheel_length+width)/2} ${wheel_radius}"/>
+    <parent link="${car_name}/base_link"/>
+    <child link="${car_name}/back_right_wheel"/>
+    <origin xyz="0 ${-(wheel_length+width)/2} ${wheel_radius}"/>
   </joint>
-  <link name="back_right_wheel">
+  <link name="${car_name}/back_right_wheel">
     <visual>
       <geometry>
@@ -68,14 +69,14 @@
   </link>
   <joint name="base_to_front_left_hinge" type="fixed">
-    <parent link="base_link"/>
-    <child link="front_left_hinge"/>
-    <origin xyz="${wheelbase/2-0.1} ${(wheel_length+width)/2} ${wheel_radius}"/>
+    <parent link="${car_name}/base_link"/>
+    <child link="${car_name}/front_left_hinge"/>
+    <origin xyz="${wheelbase} ${(wheel_length+width)/2} ${wheel_radius}"/>
   </joint>
-  <link name="front_left_hinge"/>
+  <link name="${car_name}/front_left_hinge"/>
   <joint name="front_left_hinge_to_wheel" type="continuous">
-    <parent link="front_left_hinge"/>
-    <child link="front_left_wheel"/>
+    <parent link="${car_name}/front_left_hinge"/>
+    <child link="${car_name}/front_left_wheel"/>
   </joint>
-  <link name="front_left_wheel">
+  <link name="${car_name}/front_left_wheel">
     <visual>
       <geometry>
@@ -87,14 +88,14 @@
   </link>
   <joint name="base_to_front_right_hinge" type="fixed">
-    <parent link="base_link"/>
-    <child link="front_right_hinge"/>
-    <origin xyz="${wheelbase/2-0.1} ${-(wheel_length+width)/2} ${wheel_radius}"/>
+    <parent link="${car_name}/base_link"/>
+    <child link="${car_name}/front_right_hinge"/>
+    <origin xyz="${wheelbase} ${-(wheel_length+width)/2} ${wheel_radius}"/>
   </joint>
-  <link name="front_right_hinge"/>
+  <link name="${car_name}/front_right_hinge"/>
   <joint name="front_right_hinge_to_wheel" type="continuous">
-    <parent link="front_right_hinge"/>
-    <child link="front_right_wheel"/>
+    <parent link="${car_name}/front_right_hinge"/>
+    <child link="${car_name}/front_right_wheel"/>
   </joint>
-  <link name="front_right_wheel">
+  <link name="${car_name}/front_right_wheel">
     <visual>
       <geometry>
